Commit message: a robot test script for moveit, and updated urdf files

File: mnist_publisher/urdf/mrm.xacro (robot description, xacro)
@@ -76,9 +76,57 @@
   <link name="link4">
       <visual>
+          <origin rpy="0 0 0" xyz="0 0 0.4"/>
+          <geometry>
+              <cylinder radius="0.15" length="0.8"/>
+          </geometry>
+          <material name="blue"/>
+      </visual>
+  </link>
+    <joint name="link4__link5" type="revolute">
+      <axis xyz="0 1 0" />
+      <limit effort="1000.0" lower="-3.14" upper="3.14" velocity="0.5" />
+      <origin rpy="0 0 0" xyz="0 0 0.8"/>
+      <parent link="link4"/>
+      <child link="link5"/>
+  </joint>
+  <link name="link5">
+      <visual>
+          <origin rpy="0 0 0" xyz="0 0 0.4"/>
+          <geometry>
+              <cylinder radius="0.15" length="0.8"/>
+          </geometry>
+          <material name="blue"/>
+      </visual>
+  </link>
+    <joint name="link5__link6" type="revolute">
+      <axis xyz="0 1 0" />
+      <limit effort="1000.0" lower="-3.14" upper="3.14" velocity="0.5" />
+      <origin rpy="0 0 0" xyz="0 0 0.8"/>
+      <parent link="link5"/>
+      <child link="link6"/>
+  </joint>
+  <link name="link6">
+      <visual>
+          <origin rpy="0 0 0" xyz="0 0 0.4"/>
+          <geometry>
+              <cylinder radius="0.15" length="0.8"/>
+          </geometry>
+          <material name="blue"/>
+      </visual>
+  </link>
+    <joint name="link6__link7" type="revolute">
+      <axis xyz="0 1 0" />
+      <limit effort="1000.0" lower="-3.14" upper="3.14" velocity="0.5" />
+      <origin rpy="0 0 0" xyz="0 0 0.8"/>
+      <parent link="link6"/>
+      <child link="link7"/>
+  </joint>
+  <link name="link7">
+      <visual>
           <origin rpy="0 0 0" xyz="0 0 0.125"/>
           <geometry>
               <cylinder radius="0.15" length="0.25"/>
           </geometry>
-          <material name="white"/>
+          <material name="blue"/>
       </visual>
   </link>

Commit message: launch files for rviz, working urdf, mnist trajectory

File: mnist_publisher/urdf/mrm.xacro (robot description, xacro)
@@ -24,19 +24,19 @@
       <child link="link1"/>
   </joint>
-  <link name="link1">
+   -->
+  <link name="base_link">
       <visual>
-          <origin rpy="0 0 0" xyz="0 0 0.2"/>
+          <origin rpy="0 0 0" xyz="0 0 0.0"/>
           <geometry>
-              <cylinder radius="0.35" length="0.4"/>
+              <cylinder radius="0.35" length="0.0"/>
           </geometry>
           <material name="black"/>
       </visual>
   </link>
-    -->
-  <joint name="link1__link2" type="revolute">
+  <joint name="base_link__link2" type="revolute">
       <axis xyz="0 1 0" />
       <limit effort="1000.0" lower="-3.14" upper="3.14" velocity="0.5" />
       <origin rpy="0 0 0" xyz="0 0 0"/>
-      <parent link="link1"/>
+      <parent link="base_link"/>
       <child link="link2"/>
   </joint>

Commit message: valid orientation urdf

File: mnist_publisher/urdf/mrm.xacro (robot description, xacro)
@@ -7,25 +7,7 @@
     <color rgba="1 1 1 1"/>
   </material>
-<!--
   <link name="base_link">
       <visual>
-          <origin rpy="0 0 0" xyz="0 0 0"/>
-          <geometry>
-              <box size="1 1 1"/>
-          </geometry>
-          <material name="black"/>
-      </visual>
-  </link>
-  <joint name="base_link__link1" type="fixed">
-      <axis xyz="0 0 1" />
-      <limit effort="1000.0" lower="-3.14" upper="3.14" velocity="0.5" />
-      <origin rpy="0 0 0" xyz="0 0 0.5"/>
-      <parent link="base_link"/>
-      <child link="link1"/>
-  </joint>
-   -->
-  <link name="base_link">
-      <visual>
-          <origin rpy="0 0 0" xyz="0 0 0.0"/>
+          <origin rpy="1.575 0 0" xyz="0 0 0.0"/>
           <geometry>
               <cylinder radius="0.35" length="0.0"/>
@@ -35,5 +17,5 @@
   </link>
   <joint name="base_link__link2" type="revolute">
-      <axis xyz="0 1 0" />
+      <axis xyz="0 0 1" />
       <limit effort="1000.0" lower="-3.14" upper="3.14" velocity="0.5" />
       <origin rpy="0 0 0" xyz="0 0 0"/>
@@ -43,5 +25,5 @@
   <link name="link2">
       <visual>
-          <origin rpy="0 0 0" xyz="0 0 0.4"/>
+          <origin rpy="1.575 0 0" xyz="0 0.4 0"/>
           <geometry>
               <cylinder radius="0.15" length="0.8"/>
@@ -60,7 +42,7 @@
   </link>
   <joint name="link2__link3" type="revolute">
-      <axis xyz="0 1 0" />
+      <axis xyz="0 0 1" />
       <limit effort="1000.0" lower="-3.14" upper="3.14" velocity="0.5" />
-      <origin rpy="0 0 0" xyz="0 0 0.8"/>
+      <origin rpy="0 0 0" xyz="0 0.8 0"/>
       <parent link="link2"/>
       <child link="link3"/>
@@ -68,5 +50,5 @@
   <link name="link3">
       <visual>
-          <origin rpy="0 0 0" xyz="0 0 0.4"/>
+          <origin rpy="1.575 0 0" xyz="0 0.4 0"/>
           <geometry>
               <cylinder radius="0.15" length="0.8"/>
