Commit message: fix naming of joints in .xacro file and in mover.py to allow for joint_State messages to be published

File: urdf/mrm.xacro (robot description, xacro)
@@ -16,5 +16,5 @@
       </visual>
   </link>
-  <joint name="base_link__link2" type="revolute">
+  <joint name="joint0" type="revolute">
       <axis xyz="0 0 1" />
       <limit effort="1000.0" lower="-3.14" upper="3.14" velocity="0.5" />
@@ -41,5 +41,5 @@
       </inertial>
   </link>
-  <joint name="link2__link3" type="revolute">
+  <joint name="joint1" type="revolute">
       <axis xyz="0 0 1" />
       <limit effort="1000.0" lower="-3.14" upper="3.14" velocity="0.5" />
